Commit message: add hinged door

File: dor_description/urdf/triwheeler.urdf.xacro (robot description, xacro)
@@ -2,5 +2,5 @@
 <robot xmlns:xacro="https://www.ros.org/wiki/xacro" >
     <xacro:property name="PI" value="3.1415926535897931"/>
-    <xacro:property name="chassis_x" value="0.6" />
+    <xacro:property name="chassis_x" value="0.4" />
     <xacro:property name="chassis_y" value="0.4" />
     <xacro:property name="chassis_z" value="0.2" />
@@ -11,5 +11,5 @@
     <xacro:property name="caster_r" value="0.1"/>
     <xacro:property name="caster_m" value="0.1"/>
-    <xacro:property name="wheelbase" value="0.6" />
+    <xacro:property name="wheelbase" value="0.4" />
     <xacro:property name="track" value="0.48" />
     <!-- main triwheeler link -->
