Commit message: remove bar slider as it will cause the robot crash

File: dor_description/urdf/operate_device.urdf.xacro (robot description, xacro)
@@ -30,10 +30,12 @@
         </inertial>
       </link>
-      <joint name="joint_bar_slider1" type="prismatic">
+      <!--joint name="joint_bar_slider1" type="prismatic" have an issue-->
+      <joint name="joint_bar_slider1" type="fixed">
         <origin xyz="0.02 0 0" rpy="0 0 0"/>
         <parent link="link_bar"/>
         <child link="link_slider1"/>
         <axis xyz="0 1 0"/>
-        <limit upper="0.15" lower="-0.15" effort="30.0" velocity="0.1"/>
+        <limit upper="0.15" lower="-0.15" effort="100.0" velocity="0.1"/>
+        <dynamics damping="0" friction="0"/>
       </joint>
       <link name="link_slider1">
@@ -130,5 +132,5 @@
         </inertial>
       </link>
-      <transmission name="bar_trans">
+      <!--transmission name="bar_trans">
         <type>transmission_interface/SimpleTransmission</type>
         <joint name="joint_bar_slider1">
@@ -139,5 +141,5 @@
           <mechanicalReduction>1</mechanicalReduction>
         </actuator>
-      </transmission>
+      </transmission-->
       <transmission name="lift_trans">
         <type>transmission_interface/SimpleTransmission</type>

Commit message: add hook

File: dor_description/urdf/operate_device.urdf.xacro (robot description, xacro)
@@ -25,4 +25,8 @@
     <xacro:property name="tip_z" value="0.06" />
     <xacro:property name="tip_m" value="0.01" />
+    <xacro:property name="hook_x" value="0.15" />
+    <xacro:property name="hook_y" value="0.02" />
+    <xacro:property name="hook_z" value="0.02" />
+    <xacro:property name="hook_m" value="0.01" />
     <xacro:macro name="operate_device_macro" params="parent robotname">
       <joint name="joint_support_bar" type="fixed">
@@ -152,4 +156,31 @@
         </inertial>
       </link>
+      <!--hook for opening door-->
+      <joint name="joint_bar_hook" type="revolute">
+        <origin xyz="${bar_x/2} ${bar_y/2} 0.1" rpy="0 0 0"/>
+        <parent link="link_bar"/>
+        <child link="link_hook"/>
+        <axis xyz="0 1 0"/>
+        <limit effort="30.0" lower="0.0" upper="1.57" velocity="0.5"/>
+      </joint>
+      <link name="link_hook">
+        <visual>
+          <origin xyz="${hook_x/2} ${hook_y/2} 0" rpy="0 0 0" />
+          <geometry>
+            <box size="${hook_x} ${hook_y} ${hook_z}"/>
+          </geometry>
+        </visual>
+        <collision>
+          <origin xyz="${hook_x/2} ${hook_y/2} 0" rpy="0 0 0" />
+          <geometry>
+            <box size="${hook_x} ${hook_y} ${hook_z}"/>
+          </geometry>
+        </collision>
+        <inertial>
+          <mass value="${hook_m}"/>
+          <origin xyz="${hook_x/2} ${hook_y/2} 0" rpy="0 0 0" />
+          <inertia ixx="${1/12*hook_m*(hook_y*hook_y+hook_z*hook_z)}" ixy="0" ixz="0" iyy="${1/12*hook_m*(hook_z*hook_z+hook_x*hook_x)}" iyz="0" izz="${1/12*hook_m*(hook_x*hook_x+hook_y*hook_y)}"/>
+        </inertial>
+      </link>
       <transmission name="vertical_trans">
         <type>transmission_interface/SimpleTransmission</type>
@@ -172,16 +203,25 @@
         </actuator>
       </transmission>
+      <transmission name="hook_trans">
+        <type>transmission_interface/SimpleTransmission</type>
+        <joint name="joint_bar_hook">
+          <hardwareInterface>EffortJointInterface</hardwareInterface>
+        </joint>
+        <actuator name="hook_motor">
+          <hardwareInterface>EffortJointInterface</hardwareInterface>
+          <mechanicalReduction>1</mechanicalReduction>
+        </actuator>
+      </transmission>
       <gazebo reference="link_bar">
         <material>Gazebo/Orange</material>
-        <!-- <selfCollide>false</selfCollide> -->
       </gazebo>
       <gazebo reference="link_vslider">
         <material>Gazebo/Orange</material>
-        <!-- <selfCollide>false</selfCollide> -->
-        <!-- <turnOnGravity>false</turnOnGravity> -->
       </gazebo>
       <gazebo reference="link_hslider">
         <material>Gazebo/Orange</material>
-        <!-- <selfCollide>false</selfCollide> -->
+      </gazebo>
+      <gazebo reference="link_hook">
+        <material>Gazebo/Black</material>
       </gazebo>
       <gazebo>
