Commit message: add joint control

File: dor_description/urdf/mobile_robot.urdf.xacro (robot description, xacro)
@@ -2,4 +2,21 @@
 <robot name="mobile_robot" xmlns:xacro="https://www.ros.org/wiki/xacro" >
     <xacro:include filename="$(find dor_description)/urdf/triwheeler.urdf.xacro" />
-    <xacro:triwheeler_base_macro />
+    <xacro:triwheeler_base_macro>
+      <xacro:property name="chassis_x" value="0.6" />
+      <xacro:property name="chassis_y" value="0.4" />
+      <xacro:property name="chassis_z" value="0.2" />
+      <xacro:property name="support_x" value="0.6" />
+      <xacro:property name="support_y" value="0.4" />
+      <xacro:property name="support_z" value="0.6" />
+      <xacro:property name="wheel_r" value="0.2"/>
+      <xacro:property name="wheel_l" value="0.08"/>
+      <xacro:property name="wheelbase" value="0.5" />
+      <xacro:property name="track" value="0.48" />
+    </xacro:triwheeler_base_macro>
+    <xacro:include filename="$(find dor_description)/urdf/operate_device.urdf.xacro" />
+    <xacro:operate_device_macro parent="link_support" robotname="mobile_robot">
+      <xacro:property name="location_x" value="0.3" />
+      <xacro:property name="location_y" value="0" />
+      <xacro:property name="location_z" value="0.45" />
+    </xacro:operate_device_macro>
 </robot>

File: dor_description/urdf/triwheeler.urdf.xacro (robot description, xacro)
@@ -5,5 +5,5 @@
     <xacro:property name="chassis_y" value="0.4" />
     <xacro:property name="chassis_z" value="0.2" />
-    <xacro:property name="chassis_m" value="20" />
+    <xacro:property name="chassis_m" value="30" />
     <xacro:property name="wheel_r" value="0.2"/>
     <xacro:property name="wheel_l" value="0.08"/>
@@ -11,6 +11,10 @@
     <xacro:property name="caster_r" value="0.1"/>
     <xacro:property name="caster_m" value="0.1"/>
-    <xacro:property name="wheelbase" value="0.4" />
-    <xacro:property name="track" value="0.48" />
+    <xacro:property name="wheelbase" value="0.3" />
+    <xacro:property name="track" value="0.38" />
+    <xacro:property name="support_x" value="0.4" />
+    <xacro:property name="support_y" value="0.4" />
+    <xacro:property name="support_z" value="1.0" />
+    <xacro:property name="support_m" value="1" />
     <!-- main triwheeler link -->
     <xacro:macro name="triwheeler_base_macro">
@@ -25,5 +29,5 @@
           <origin xyz="0 0 0" rpy="0 0 0" />
           <geometry>
-            <box size="${chassis_x} ${chassis_y} ${chassis_z}"/> />
+            <box size="${chassis_x} ${chassis_y} ${chassis_z}"/>
           </geometry>
         </visual>
@@ -31,5 +35,5 @@
           <origin xyz="0 0 0" rpy="0 0 0" />
           <geometry>
-            <box size="${chassis_x} ${chassis_y} ${chassis_z}"/> />
+            <box size="${chassis_x} ${chassis_y} ${chassis_z}"/>
           </geometry>
         </collision>
@@ -114,4 +118,28 @@
         </inertial>
       </link>
+      <joint name="joint_chassis_support" type="fixed">
+        <origin rpy="0 0 0" xyz="0 0 ${chassis_z/2}"/>
+        <parent link="link_chassis"/>
+        <child link="link_support"/>
+      </joint>
+      <link name="link_support">
+        <visual>
+          <origin xyz="0 0 ${support_z/2}" rpy="0 0 0" />
+          <geometry>
+            <box size="${support_x} ${support_y} ${support_z}"/>
+          </geometry>
+        </visual>
+        <collision>
+          <origin xyz="0 0 ${support_z/2}" rpy="0 0 0" />
+          <geometry>
+            <box size="${support_x} ${support_y} ${support_z}"/>
+          </geometry>
+        </collision>
+        <inertial>
+          <mass value="${support_m}"/>
+          <origin rpy="0 0 0" xyz="0 0 0"/>
+          <inertia ixx="${1/12*support_m*(support_y*support_y+support_z*support_z)}" ixy="0" ixz="0" iyy="${1/12*support_m*(support_z*support_z+support_x*support_x)}" iyz="0" izz="${1/12*support_m*(support_x*support_x+support_y*support_y)}"/>
+        </inertial>
+      </link>
       <!--Gazebo-->
       <!-- differential_drive_controller -->
@@ -125,5 +153,5 @@
           <wheelSeparation>${chassis_y}+${wheel_l}</wheelSeparation>
           <wheelDiameter>2*${wheel_r}</wheelDiameter>
-          <wheelTorque>1</wheelTorque>
+          <wheelTorque>90</wheelTorque>
           <!--wheelAcceleration>${wheel_accel}</wheelAcceleration-->
           <commandTopic>cmd_vel</commandTopic>

Commit message: add camera

File: dor_description/urdf/mobile_robot.urdf.xacro (robot description, xacro)
@@ -1,6 +1,6 @@
 <?xml version="1.0"?>
 <robot name="mobile_robot" xmlns:xacro="https://www.ros.org/wiki/xacro" >
-    <xacro:include filename="$(find dor_description)/urdf/triwheeler.urdf.xacro" />
-    <xacro:triwheeler_base_macro>
+    <xacro:include filename="$(find dor_description)/urdf/fourwheeler.urdf.xacro" />
+    <xacro:fourwheeler_base_macro>
       <xacro:property name="chassis_x" value="0.6" />
       <xacro:property name="chassis_y" value="0.4" />
@@ -9,14 +9,24 @@
       <xacro:property name="support_y" value="0.4" />
       <xacro:property name="support_z" value="0.6" />
-      <xacro:property name="wheel_r" value="0.2"/>
+      <xacro:property name="wheel_r" value="0.15"/>
       <xacro:property name="wheel_l" value="0.08"/>
-      <xacro:property name="wheelbase" value="0.5" />
+      <xacro:property name="wheelbase" value="0.4" />
       <xacro:property name="track" value="0.48" />
-    </xacro:triwheeler_base_macro>
+    </xacro:fourwheeler_base_macro>
     <xacro:include filename="$(find dor_description)/urdf/operate_device.urdf.xacro" />
     <xacro:operate_device_macro parent="link_support" robotname="mobile_robot">
       <xacro:property name="location_x" value="0.3" />
       <xacro:property name="location_y" value="0" />
-      <xacro:property name="location_z" value="0.45" />
+      <xacro:property name="location_z" value="0.5" />
     </xacro:operate_device_macro>
+    <xacro:include filename="$(find dor_description)/urdf/camera.urdf.xacro"/>
+    <xacro:camera_macro parent="link_support">
+      <xacro:property name="location_x" value="0.2" />
+      <xacro:property name="location_y" value="0" />
+      <xacro:property name="location_z" value="0.3" />
+      <xacro:property name="support_x" value="0.02"/>
+      <xacro:property name="support_y" value="0.02"/>
+      <xacro:property name="support_z" value="0.8"/>
+      <xacro:property name="support_m" value="0.5"/>
+    </xacro:camera_macro>
 </robot>

Commit message: add laser support

File: dor_description/urdf/mobile_robot.urdf.xacro (robot description, xacro)
@@ -30,3 +30,9 @@
       <xacro:property name="support_m" value="0.5"/>
     </xacro:camera_macro>
+    <xacro:include filename="$(find dor_description)/urdf/laser.urdf.xacro"/>
+    <xacro:laser_macro parent="link_chassis">
+      <xacro:property name="location_x" value="0.35" />
+      <xacro:property name="location_y" value="0" />
+      <xacro:property name="location_z" value="0" />
+    </xacro:laser_macro>
 </robot>

Commit message: fix the hook issue with correct inertia

File: dor_description/urdf/mobile_robot.urdf.xacro (robot description, xacro)
@@ -8,5 +8,5 @@
       <xacro:property name="location_x" value="0.25" />
       <xacro:property name="location_y" value="0" />
-      <xacro:property name="location_z" value="0.5" />
+      <xacro:property name="location_z" value="0.55" />
     </xacro:operate_device_macro>
     <xacro:include filename="$(find dor_description)/urdf/camera.urdf.xacro"/>

File: dor_description/urdf/operate_device.urdf.xacro (robot description, xacro)
@@ -10,5 +10,5 @@
     <xacro:property name="bar_m" value="0.5" />
     <xacro:property name="vslider_x" value="0.02" />
-    <xacro:property name="vslider_y" value="0.5" />
+    <xacro:property name="vslider_y" value="0.2" />
     <xacro:property name="vslider_z" value="0.05" />
     <xacro:property name="vslider_m" value="0.2" />
@@ -25,7 +25,6 @@
     <xacro:property name="tip_z" value="0.06" />
     <xacro:property name="tip_m" value="0.01" />
-    <xacro:property name="hook_x" value="0.15" />
-    <xacro:property name="hook_y" value="0.02" />
-    <xacro:property name="hook_z" value="0.02" />
+    <xacro:property name="hook_l" value="0.2" />
+    <xacro:property name="hook_r" value="0.01" />
     <xacro:property name="hook_m" value="0.01" />
     <xacro:macro name="operate_device_macro" params="parent robotname">
@@ -59,6 +58,6 @@
         <child link="link_vslider"/>
         <axis xyz="0 0 1"/>
-        <limit upper="${bar_z-0.05}" lower="0.0" effort="100.0" velocity="0.5"/>
-        <!-- <dynamics damping="0" friction="0.2"/> -->
+        <limit upper="${bar_z-0.05}" lower="0.0" effort="1000.0" velocity="0.5"/>
+        <dynamics damping="0" friction="1.0"/>
       </joint>
       <link name="link_vslider">
@@ -86,6 +85,6 @@
         <child link="link_hslider"/>
         <axis xyz="0 1 0"/>
-        <limit upper="0.225" lower="-0.225" effort="100.0" velocity="0.5"/>
-        <!-- <dynamics damping="0" friction="0.2"/> -->
+        <limit upper="0.225" lower="-0.225" effort="1000.0" velocity="0.5"/>
+        <dynamics damping="0" friction="1.0"/>
       </joint>
       <link name="link_hslider">
@@ -158,29 +157,40 @@
       <!--hook for opening door-->
       <joint name="joint_bar_hook" type="revolute">
-        <origin xyz="${bar_x/2} ${bar_y/2} 0.1" rpy="0 0 0"/>
+        <origin xyz="${bar_x/2} ${bar_y/2} 0" rpy="0 0 0"/>
         <parent link="link_bar"/>
         <child link="link_hook"/>
         <axis xyz="0 1 0"/>
-        <limit effort="30.0" lower="0.0" upper="1.57" velocity="0.5"/>
+        <limit effort="1000.0" lower="0.0" upper="${0.5*PI}" velocity="0.5"/>
+        <dynamics damping="0" friction="1.0"/>
       </joint>
       <link name="link_hook">
         <visual>
-          <origin xyz="${hook_x/2} ${hook_y/2} 0" rpy="0 0 0" />
-          <geometry>
-            <box size="${hook_x} ${hook_y} ${hook_z}"/>
-          </geometry>
-        </visual>
-        <collision>
-          <origin xyz="${hook_x/2} ${hook_y/2} 0" rpy="0 0 0" />
-          <geometry>
-            <box size="${hook_x} ${hook_y} ${hook_z}"/>
+          <origin xyz="${hook_r} ${hook_r} ${hook_l/2}" rpy="0 0 0" />
+          <geometry>
+            <cylinder length="${hook_l}" radius="${hook_r}"/>
+          </geometry>
+        </visual>
+        <collision>
+          <origin xyz="${hook_r} ${hook_r} ${hook_l/2}" rpy="0 0 0" />
+          <geometry>
+            <cylinder length="${hook_l}" radius="${hook_r}"/>
           </geometry>
         </collision>
         <inertial>
           <mass value="${hook_m}"/>
-          <origin xyz="${hook_x/2} ${hook_y/2} 0" rpy="0 0 0" />
-          <inertia ixx="${1/12*hook_m*(hook_y*hook_y+hook_z*hook_z)}" ixy="0" ixz="0" iyy="${1/12*hook_m*(hook_z*hook_z+hook_x*hook_x)}" iyz="0" izz="${1/12*hook_m*(hook_x*hook_x+hook_y*hook_y)}"/>
-        </inertial>
-      </link>
+          <origin xyz="${hook_r} ${hook_r} ${hook_l/2}" rpy="0 0 0" />
+          <inertia ixx="${1/3*hook_m*hook_l*hook_l}" ixy="0" ixz="0" iyy="0" iyz="0" izz="${1/3*hook_m*hook_l*hook_l}"/>
+        </inertial>
+      </link>
+      <transmission name="hook_trans">
+        <type>transmission_interface/SimpleTransmission</type>
+        <joint name="joint_bar_hook">
+          <hardwareInterface>EffortJointInterface</hardwareInterface>
+        </joint>
+        <actuator name="hook_motor">
+          <hardwareInterface>EffortJointInterface</hardwareInterface>
+          <mechanicalReduction>1</mechanicalReduction>
+        </actuator>
+      </transmission>
       <transmission name="vertical_trans">
         <type>transmission_interface/SimpleTransmission</type>
@@ -203,14 +213,4 @@
         </actuator>
       </transmission>
-      <transmission name="hook_trans">
-        <type>transmission_interface/SimpleTransmission</type>
-        <joint name="joint_bar_hook">
-          <hardwareInterface>EffortJointInterface</hardwareInterface>
-        </joint>
-        <actuator name="hook_motor">
-          <hardwareInterface>EffortJointInterface</hardwareInterface>
-          <mechanicalReduction>1</mechanicalReduction>
-        </actuator>
-      </transmission>
       <gazebo reference="link_bar">
         <material>Gazebo/Orange</material>
@@ -218,10 +218,13 @@
       <gazebo reference="link_vslider">
         <material>Gazebo/Orange</material>
+        <turnGravityOff>false</turnGravityOff>
       </gazebo>
       <gazebo reference="link_hslider">
         <material>Gazebo/Orange</material>
+        <turnGravityOff>false</turnGravityOff>
       </gazebo>
       <gazebo reference="link_hook">
         <material>Gazebo/Black</material>
+        <turnGravityOff>false</turnGravityOff>
       </gazebo>
       <gazebo>
