Commit message: fix prismatic joint break issue with making the limit range positive

File: dor_description/urdf/fourwheeler.urdf.xacro (robot description, xacro)
@@ -5,5 +5,5 @@
     <xacro:property name="chassis_y" value="0.4" />
     <xacro:property name="chassis_z" value="0.05" />
-    <xacro:property name="chassis_m" value="8" />
+    <xacro:property name="chassis_m" value="28" />
     <xacro:property name="wheel_r" value="0.075"/>
     <xacro:property name="wheel_l" value="0.05"/>
@@ -22,5 +22,5 @@
     <xacro:property name="support_y" value="0.5" />
     <xacro:property name="support_z" value="0.5" />
-    <xacro:property name="support_m" value="26" />
+    <xacro:property name="support_m" value="6" />
     <!-- main triwheeler link -->
     <xacro:macro name="fourwheeler_base_macro">

File: dor_description/urdf/operate_device.urdf.xacro (robot description, xacro)
@@ -7,14 +7,22 @@
     <xacro:property name="bar_x" value="0.02" />
     <xacro:property name="bar_y" value="0.2" />
-    <xacro:property name="bar_z" value="1.0" />
-    <xacro:property name="bar_m" value="0.1" />
+    <xacro:property name="bar_z" value="1.05" />
+    <xacro:property name="bar_m" value="0.5" />
     <xacro:property name="vslider_x" value="0.02" />
     <xacro:property name="vslider_y" value="0.5" />
     <xacro:property name="vslider_z" value="0.05" />
-    <xacro:property name="vslider_m" value="0.1" />
+    <xacro:property name="vslider_m" value="0.2" />
     <xacro:property name="hslider_x" value="0.02" />
     <xacro:property name="hslider_y" value="0.05" />
     <xacro:property name="hslider_z" value="0.05" />
     <xacro:property name="hslider_m" value="0.1" />
+    <xacro:property name="finger_x" value="0.1" />
+    <xacro:property name="finger_y" value="0.02" />
+    <xacro:property name="finger_z" value="0.02" />
+    <xacro:property name="finger_m" value="0.01" />
+    <xacro:property name="tip_x" value="0.01" />
+    <xacro:property name="tip_y" value="0.02" />
+    <xacro:property name="tip_z" value="0.06" />
+    <xacro:property name="tip_m" value="0.01" />
     <xacro:macro name="operate_device_macro" params="parent robotname">
       <joint name="joint_support_bar" type="fixed">
@@ -43,10 +51,10 @@
       </link>
       <joint name="joint_bar_vslider" type="prismatic">
-        <origin xyz="${bar_x} 0 0" rpy="0 0 0"/>
+        <origin xyz="${bar_x} 0 -${bar_z/2}" rpy="0 0 0"/>
         <parent link="link_bar"/>
         <child link="link_vslider"/>
         <axis xyz="0 0 1"/>
-        <limit upper="0.9" lower="-0.4" effort="100.0" velocity="1.0"/>
-        <dynamics damping="1.0" friction="30.0"/>
+        <limit upper="${bar_z-0.05}" lower="0.0" effort="100.0" velocity="0.5"/>
+        <!-- <dynamics damping="0" friction="0.2"/> -->
       </joint>
       <link name="link_vslider">
@@ -69,5 +77,5 @@
         </inertial>
       </link>
-      <joint name="joint_slider_slider" type="fixed">
+      <joint name="joint_slider_slider" type="prismatic">
         <origin xyz="${vslider_x} 0 0" rpy="0 0 0"/>
         <parent link="link_vslider"/>
@@ -75,5 +83,5 @@
         <axis xyz="0 1 0"/>
         <limit upper="0.225" lower="-0.225" effort="100.0" velocity="0.5"/>
-        <dynamics damping="1.0" friction="30.0"/>
+        <!-- <dynamics damping="0" friction="0.2"/> -->
       </joint>
       <link name="link_hslider">
@@ -103,23 +111,23 @@
       <link name="link_finger">
         <visual>
-          <origin xyz="0.05 0 0" rpy="0 0 0" />
+          <origin xyz="${finger_x/2} 0 0" rpy="0 0 0" />
           <geometry>
-            <box size="0.1 0.02 0.02"/>
+            <box size="${finger_x} ${finger_y} ${finger_z}"/>
           </geometry>
         </visual>
         <collision>
-          <origin xyz="0.05 0 0" rpy="0 0 0" />
+          <origin xyz="${finger_x/2} 0 0" rpy="0 0 0" />
           <geometry>
-            <box size="0.1 0.02 0.02"/>
+            <box size="${finger_x} ${finger_y} ${finger_z}"/>
           </geometry>
         </collision>
         <inertial>
-          <mass value="0.02"/>
-          <origin xyz="0.05 0 0" rpy="0 0 0" />
-          <inertia ixx="0.000001" ixy="0" ixz="0" iyy="0.000017" iyz="0" izz="0.000017"/>
+          <mass value="${finger_m}"/>
+          <origin xyz="${finger_x/2} 0 0" rpy="0 0 0" />
+          <inertia ixx="${1/12*finger_m*(finger_y*finger_y+finger_z*finger_z)}" ixy="0" ixz="0" iyy="${1/12*finger_m*(finger_z*finger_z+finger_x*finger_x)}" iyz="0" izz="${1/12*finger_m*(finger_x*finger_x+finger_y*finger_y)}"/>
         </inertial>
       </link>
       <joint name="joint_finger_tip" type="fixed">
-        <origin xyz="0.1 0 0" rpy="0 0 0"/>
+        <origin xyz="${finger_x} 0 0" rpy="0 0 0"/>
         <parent link="link_finger"/>
         <child link="link_tip"/>
@@ -127,19 +135,19 @@
       <link name="link_tip">
         <visual>
-          <origin xyz="0.005 0 -0.015" rpy="0 0 0" />
+          <origin xyz="${tip_x/2} 0 -0.02" rpy="0 0 0" />
           <geometry>
-            <box size="0.01 0.02 0.05"/>
+            <box size="${tip_x} ${tip_y} ${tip_z}"/>
           </geometry>
         </visual>
         <collision>
-          <origin xyz="0.005 0 -0.015" rpy="0 0 0" />
+          <origin xyz="${tip_x/2} 0 -0.02" rpy="0 0 0" />
           <geometry>
-            <box size="0.01 0.02 0.05"/>
+            <box size="${tip_x} ${tip_y} ${tip_z}"/>
           </geometry>
         </collision>
         <inertial>
-          <mass value="0.001"/>
-          <origin xyz="0.005 0 -0.015" rpy="0 0 0" />
-          <inertia ixx="0.00000001" ixy="0" ixz="0" iyy="0.000000017" iyz="0" izz="0.0000000017"/>
+          <mass value="${tip_m}"/>
+          <origin xyz="${tip_x/2} 0 -0.02" rpy="0 0 0" />
+          <inertia ixx="${1/12*tip_m*(tip_y*tip_y+tip_z*tip_z)}" ixy="0" ixz="0" iyy="${1/12*tip_m*(tip_z*tip_z+tip_x*tip_x)}" iyz="0" izz="${1/12*tip_m*(tip_x*tip_x+tip_y*tip_y)}"/>
         </inertial>
       </link>
@@ -154,5 +162,5 @@
         </actuator>
       </transmission>
-      <!-- <transmission name="horizontal_trans">
+      <transmission name="horizontal_trans">
         <type>transmission_interface/SimpleTransmission</type>
         <joint name="joint_slider_slider">
@@ -163,13 +171,17 @@
           <mechanicalReduction>1</mechanicalReduction>
         </actuator>
-      </transmission> -->
+      </transmission>
       <gazebo reference="link_bar">
         <material>Gazebo/Orange</material>
+        <!-- <selfCollide>false</selfCollide> -->
       </gazebo>
       <gazebo reference="link_vslider">
         <material>Gazebo/Orange</material>
+        <!-- <selfCollide>false</selfCollide> -->
+        <!-- <turnOnGravity>false</turnOnGravity> -->
       </gazebo>
       <gazebo reference="link_hslider">
         <material>Gazebo/Orange</material>
+        <!-- <selfCollide>false</selfCollide> -->
       </gazebo>
       <gazebo>

Commit message: door opening demo

File: dor_description/urdf/fourwheeler.urdf.xacro (robot description, xacro)
@@ -23,4 +23,7 @@
     <xacro:property name="support_z" value="0.5" />
     <xacro:property name="support_m" value="6" />
+    <xacro:property name="hook_l" value="0.25" />
+    <xacro:property name="hook_r" value="0.01" />
+    <xacro:property name="hook_m" value="0.01" />
     <!-- main triwheeler link -->
     <xacro:macro name="fourwheeler_base_macro">
@@ -252,4 +255,66 @@
         </inertial>
       </link>
+      <!--hook for opening door-->
+      <joint name="joint_support_hook" type="revolute">
+        <origin xyz="${support_x/2} ${support_y/2} 0" rpy="0 0 0"/>
+        <parent link="link_support"/>
+        <child link="link_hook"/>
+        <axis xyz="0 1 0"/>
+        <limit effort="1000.0" lower="0.0" upper="${0.5*PI}" velocity="0.5"/>
+        <dynamics damping="0" friction="1.0"/>
+      </joint>
+      <link name="link_hook">
+        <visual>
+          <origin xyz="${hook_r} ${hook_r} ${hook_l/2}" rpy="0 0 0" />
+          <geometry>
+            <cylinder length="${hook_l}" radius="${hook_r}"/>
+          </geometry>
+        </visual>
+        <collision>
+          <origin xyz="${hook_r} ${hook_r} ${hook_l/2}" rpy="0 0 0" />
+          <geometry>
+            <cylinder length="${hook_l}" radius="${hook_r}"/>
+          </geometry>
+        </collision>
+        <inertial>
+          <mass value="${hook_m}"/>
+          <origin xyz="${hook_r} ${hook_r} ${hook_l/2}" rpy="0 0 0" />
+          <inertia ixx="${1/3*hook_m*hook_l*hook_l}" ixy="0" ixz="0" iyy="0" iyz="0" izz="${1/3*hook_m*hook_l*hook_l}"/>
+        </inertial>
+      </link>
+      <!-- <joint name="joint_hook_tip" type="fixed">
+        <origin xyz="${hook_r} ${hook_r} ${hook_l}" rpy="0 0 0"/>
+        <parent link="link_hook"/>
+        <child link="link_hooktip"/>
+      </joint>
+      <link name="link_hooktip">
+        <visual>
+          <origin xyz="0 0 0.015" rpy="0 0 0" />
+          <geometry>
+            <box size="0.03 0.03 0.03"/>
+          </geometry>
+        </visual>
+        <collision>
+          <origin xyz="0 0 0.01" rpy="0 0 0" />
+          <geometry>
+            <box size="0.03 0.03 0.03"/>
+          </geometry>
+        </collision>
+        <inertial>
+          <mass value="0.001"/>
+          <origin xyz="0.03 0.03 0.03" rpy="0 0 0" />
+          <inertia ixx="1e-7" ixy="0" ixz="0" iyy="1e-7" iyz="0" izz="1e-7"/>
+        </inertial>
+      </link> -->
+      <transmission name="hook_trans">
+        <type>transmission_interface/SimpleTransmission</type>
+        <joint name="joint_support_hook">
+          <hardwareInterface>hardware_interface/EffortJointInterface</hardwareInterface>
+        </joint>
+        <actuator name="hook_motor">
+          <hardwareInterface>hardware_interface/EffortJointInterface</hardwareInterface>
+          <mechanicalReduction>1</mechanicalReduction>
+        </actuator>
+      </transmission>
       <!--Gazebo-->
       <!-- skid steering controller -->
@@ -299,4 +364,8 @@
         <material>Gazebo/Black</material>
       </gazebo>
+      <gazebo reference="link_hook">
+        <material>Gazebo/Black</material>
+        <turnGravityOff>true</turnGravityOff>
+      </gazebo>
     </xacro:macro>
 </robot>

File: dor_description/urdf/laser.urdf.xacro (robot description, xacro)
@@ -37,5 +37,5 @@
           <pose>0 0 0 0 0 0</pose>
           <visualize>false</visualize>
-          <update_rate>30</update_rate>
+          <update_rate>50</update_rate>
           <ray>
             <scan>
@@ -50,10 +50,10 @@
               <min>0.01</min>
               <max>100.0</max>
-              <resolution>0.01</resolution>
+              <resolution>0.005</resolution>
             </range>
             <noise>
               <type>gaussian</type>
               <mean>0.0</mean>
-              <stddev>0.01</stddev>
+              <stddev>0.001</stddev>
             </noise>
           </ray>

File: dor_description/urdf/mobile_robot.urdf.xacro (robot description, xacro)
@@ -14,5 +14,5 @@
       <xacro:property name="location_x" value="0.025" />
       <xacro:property name="location_y" value="0.0" />
-      <xacro:property name="location_z" value="0.5" />
+      <xacro:property name="location_z" value="0.52" />
     </xacro:realsense_macro>
     <xacro:include filename="$(find dor_description)/urdf/camera.urdf.xacro"/>

File: dor_description/urdf/operate_device.urdf.xacro (robot description, xacro)
@@ -10,5 +10,5 @@
     <xacro:property name="bar_m" value="0.5" />
     <xacro:property name="vslider_x" value="0.02" />
-    <xacro:property name="vslider_y" value="0.2" />
+    <xacro:property name="vslider_y" value="0.5" />
     <xacro:property name="vslider_z" value="0.05" />
     <xacro:property name="vslider_m" value="0.2" />
@@ -25,7 +25,4 @@
     <xacro:property name="tip_z" value="0.06" />
     <xacro:property name="tip_m" value="0.01" />
-    <xacro:property name="hook_l" value="0.2" />
-    <xacro:property name="hook_r" value="0.01" />
-    <xacro:property name="hook_m" value="0.01" />
     <xacro:macro name="operate_device_macro" params="parent robotname">
       <joint name="joint_support_bar" type="fixed">
@@ -58,6 +55,6 @@
         <child link="link_vslider"/>
         <axis xyz="0 0 1"/>
-        <limit upper="${bar_z-0.05}" lower="0.05" effort="1000.0" velocity="0.5"/>
-        <dynamics damping="0" friction="1.0"/>
+        <limit upper="${bar_z-0.05}" lower="0.05" effort="1000.0" velocity="0.1"/>
+        <dynamics damping="0" friction="2.0"/>
       </joint>
       <link name="link_vslider">
@@ -85,6 +82,6 @@
         <child link="link_hslider"/>
         <axis xyz="0 1 0"/>
-        <limit upper="0.225" lower="-0.225" effort="1000.0" velocity="0.5"/>
-        <dynamics damping="0" friction="1.0"/>
+        <limit upper="${vslider_y/2}" lower="-${vslider_y/2}" effort="1000.0" velocity="0.1"/>
+        <dynamics damping="0" friction="2.0"/>
       </joint>
       <link name="link_hslider">
@@ -155,42 +152,4 @@
         </inertial>
       </link>
-      <!--hook for opening door-->
-      <joint name="joint_bar_hook" type="revolute">
-        <origin xyz="${bar_x/2} ${bar_y/2} 0" rpy="0 0 0"/>
-        <parent link="link_bar"/>
-        <child link="link_hook"/>
-        <axis xyz="0 1 0"/>
-        <limit effort="1000.0" lower="0.0" upper="${0.5*PI}" velocity="0.5"/>
-        <dynamics damping="0" friction="1.0"/>
-      </joint>
-      <link name="link_hook">
-        <visual>
-          <origin xyz="${hook_r} ${hook_r} ${hook_l/2}" rpy="0 0 0" />
-          <geometry>
-            <cylinder length="${hook_l}" radius="${hook_r}"/>
-          </geometry>
-        </visual>
-        <collision>
-          <origin xyz="${hook_r} ${hook_r} ${hook_l/2}" rpy="0 0 0" />
-          <geometry>
-            <cylinder length="${hook_l}" radius="${hook_r}"/>
-          </geometry>
-        </collision>
-        <inertial>
-          <mass value="${hook_m}"/>
-          <origin xyz="${hook_r} ${hook_r} ${hook_l/2}" rpy="0 0 0" />
-          <inertia ixx="${1/3*hook_m*hook_l*hook_l}" ixy="0" ixz="0" iyy="0" iyz="0" izz="${1/3*hook_m*hook_l*hook_l}"/>
-        </inertial>
-      </link>
-      <transmission name="hook_trans">
-        <type>transmission_interface/SimpleTransmission</type>
-        <joint name="joint_bar_hook">
-          <hardwareInterface>hardware_interface/EffortJointInterface</hardwareInterface>
-        </joint>
-        <actuator name="hook_motor">
-          <hardwareInterface>hardware_interface/EffortJointInterface</hardwareInterface>
-          <mechanicalReduction>1</mechanicalReduction>
-        </actuator>
-      </transmission>
       <transmission name="vertical_trans">
         <type>transmission_interface/SimpleTransmission</type>
@@ -224,8 +183,4 @@
         <turnGravityOff>false</turnGravityOff>
       </gazebo>
-      <gazebo reference="link_hook">
-        <material>Gazebo/Black</material>
-        <turnGravityOff>false</turnGravityOff>
-      </gazebo>
       <gazebo>
         <plugin name="gazebo_ros_control" filename="libgazebo_ros_control.so">

Commit message: rebuild map and replan tasks

File: dor_description/urdf/fourwheeler.urdf.xacro (robot description, xacro)
@@ -342,5 +342,17 @@
       </gazebo>
       <gazebo reference="link_chassis">
-        <material>Gazebo/White</material>
+        <material>Gazebo/Grey</material>
+      </gazebo>
+      <gazebo reference="link_support">
+        <material>Gazebo/DarkGrey</material>
+      </gazebo>
+      <gazebo reference="link_base">
+        <material>Gazebo/DarkGrey</material>
+      </gazebo>
+      <gazebo reference="link_fbumper">
+        <material>Gazebo/DarkGrey</material>
+      </gazebo>
+      <gazebo reference="link_rbumper">
+        <material>Gazebo/DarkGrey</material>
       </gazebo>
       <gazebo reference="link_lrwheel">
