Commit message: change dimension of mobile robot

File: dor_description/urdf/camera.urdf.xacro (robot description, xacro)
@@ -5,8 +5,4 @@
     <xacro:property name="location_y" value="0" />
     <xacro:property name="location_z" value="1.0" />
-    <xacro:property name="support_x" value="0.02"/>
-    <xacro:property name="support_y" value="0.02"/>
-    <xacro:property name="support_z" value="0.5"/>
-    <xacro:property name="support_m" value="0.5"/>
     <xacro:property name="realsense_d435_width" value="0.09"/>
     <xacro:property name="realsense_d435_height" value="0.025"/>
@@ -21,33 +17,8 @@
     <xacro:property name="realsense_d435_case_offset_z" value="0.0"/>
     <xacro:macro name="camera_macro" params="parent">
-      <!--camera support-->
-      <joint name="joint_camera_support" type="fixed">
-        <origin xyz="${location_x} ${location_y} ${location_z}" rpy="0 0 0"/>
-        <parent link="${parent}"/>
-        <child link="link_camera_support"/>
-      </joint>
-      <link name="link_camera_support">
-        <visual>
-          <origin xyz="0 0 ${0.5*support_z}" rpy="0 0 0" />
-          <geometry>
-            <box size="0.02 0.02 ${support_z}"/>
-          </geometry>
-        </visual>
-        <collision>
-          <origin xyz="0 0 0" rpy="0 0 0" />
-          <geometry>
-            <box size="0.02 0.02 ${support_z}"/>
-          </geometry>
-        </collision>
-        <inertial>
-          <mass value="0.5"/>
-          <origin xyz="0 0 0" rpy="0 0 0"/>
-          <inertia ixx="${1/12*support_m*(support_y*support_y+support_z*support_z)}" ixy="0" ixz="0" iyy="${1/12*support_m*(support_z*support_z+support_x*support_x)}" iyz="0" izz="${1/12*support_m*(support_x*support_x+support_y*support_y)}"/>
-        </inertial>
-      </link>
       <!--camera-->
       <joint name="joint_rs435" type="fixed">
-        <origin xyz="${support_x/2.0+realsense_d435_depth/2.0} 0 ${support_z}" rpy="0 0 0"/>
-        <parent link="link_camera_support"/>
+        <origin xyz="${location_x+realsense_d435_depth/2.0} ${location_y} ${location_z}" rpy="0 0 0"/>
+        <parent link="${parent}"/>
         <child link="link_rs435"/>
       </joint>

File: dor_description/urdf/fourwheeler.urdf.xacro (robot description, xacro)
@@ -2,17 +2,25 @@
 <robot xmlns:xacro="https://www.ros.org/wiki/xacro" >
     <xacro:property name="PI" value="3.1415926535897931"/>
-    <xacro:property name="chassis_x" value="0.4" />
+    <xacro:property name="chassis_x" value="0.42" />
     <xacro:property name="chassis_y" value="0.4" />
-    <xacro:property name="chassis_z" value="0.2" />
-    <xacro:property name="chassis_m" value="30" />
-    <xacro:property name="wheel_r" value="0.2"/>
-    <xacro:property name="wheel_l" value="0.08"/>
+    <xacro:property name="chassis_z" value="0.05" />
+    <xacro:property name="chassis_m" value="8" />
+    <xacro:property name="wheel_r" value="0.075"/>
+    <xacro:property name="wheel_l" value="0.05"/>
     <xacro:property name="wheel_m" value="0.5"/>
-    <xacro:property name="wheelbase" value="0.3" />
-    <xacro:property name="track" value="0.38" />
-    <xacro:property name="support_x" value="0.4" />
-    <xacro:property name="support_y" value="0.4" />
-    <xacro:property name="support_z" value="1.0" />
-    <xacro:property name="support_m" value="1" />
+    <xacro:property name="wheelbase" value="0.25" /> <!--base on the wheel diameter and chassis_x-->
+    <xacro:property name="track" value="0.45" /> <!--base on the wheel width and chassis_y-->
+    <xacro:property name="base_x" value="0.42" />
+    <xacro:property name="base_y" value="0.4" />
+    <xacro:property name="base_z" value="0.075" />
+    <xacro:property name="base_m" value="2" />
+    <xacro:property name="bumper_x" value="0.04" />
+    <xacro:property name="bumper_y" value="0.5" />
+    <xacro:property name="bumper_z" value="0.125" />
+    <xacro:property name="bumper_m" value="1" />
+    <xacro:property name="support_x" value="0.5" />
+    <xacro:property name="support_y" value="0.5" />
+    <xacro:property name="support_z" value="0.5" />
+    <xacro:property name="support_m" value="26" />
     <!-- main triwheeler link -->
     <xacro:macro name="fourwheeler_base_macro">
@@ -120,5 +128,5 @@
         </inertial>
       </link>
-      <!--right rear wheel-->
+      <!--right front wheel-->
       <joint name="joint_chassis_rfwheel" type="continuous">
         <origin xyz="${wheelbase/2} -${track/2} 0" rpy="0 0 0" />
@@ -146,7 +154,32 @@
         </inertial>
       </link>
-      <joint name="joint_chassis_support" type="fixed">
-        <origin rpy="0 0 0" xyz="0 0 ${chassis_z/2}"/>
-        <parent link="link_chassis"/>
+      <!--upper base-->
+      <joint name="joint_chassis_base" type="fixed">
+        <origin xyz="0 0 ${chassis_z/2}" rpy="0 0 0"/>
+        <parent link="link_chassis"/>
+        <child link="link_base"/>
+      </joint>
+      <link name="link_base">
+        <visual>
+          <origin xyz="0 0 ${base_z/2}" rpy="0 0 0" />
+          <geometry>
+            <box size="${base_x} ${base_y} ${base_z}"/>
+          </geometry>
+        </visual>
+        <collision>
+          <origin xyz="0 0 ${base_z/2}" rpy="0 0 0" />
+          <geometry>
+            <box size="${base_x} ${base_y} ${base_z}"/>
+          </geometry>
+        </collision>
+        <inertial>
+          <mass value="${base_m}"/>
+          <origin rpy="0 0 0" xyz="0 0 0"/>
+          <inertia ixx="${1/12*base_m*(base_y*base_y+base_z*base_z)}" ixy="0" ixz="0" iyy="${1/12*base_m*(base_z*base_z+base_x*base_x)}" iyz="0" izz="${1/12*base_m*(base_x*base_x+base_y*base_y)}"/>
+        </inertial>
+      </link>
+      <joint name="joint_base_support" type="fixed">
+        <origin rpy="0 0 0" xyz="0 0 ${base_z}"/>
+        <parent link="link_base"/>
         <child link="link_support"/>
       </joint>
@@ -168,4 +201,53 @@
           <origin rpy="0 0 0" xyz="0 0 0"/>
           <inertia ixx="${1/12*support_m*(support_y*support_y+support_z*support_z)}" ixy="0" ixz="0" iyy="${1/12*support_m*(support_z*support_z+support_x*support_x)}" iyz="0" izz="${1/12*support_m*(support_x*support_x+support_y*support_y)}"/>
+        </inertial>
+      </link>
+      <!--bumper-->
+      <joint name="joint_chassis_fbumper" type="fixed">
+        <origin xyz="${chassis_x/2} 0 ${(chassis_z+base_z)/2-chassis_z/2}" rpy="0 0 0"/>
+        <parent link="link_chassis"/>
+        <child link="link_fbumper"/>
+      </joint>
+      <link name="link_fbumper">
+        <visual>
+          <origin xyz="${bumper_x/2} 0 0" rpy="0 0 0" />
+          <geometry>
+            <box size="${bumper_x} ${bumper_y} ${bumper_z}"/>
+          </geometry>
+        </visual>
+        <collision>
+          <origin xyz="${bumper_x/2} 0 0" rpy="0 0 0" />
+          <geometry>
+            <box size="${bumper_x} ${bumper_y} ${bumper_z}"/>
+          </geometry>
+        </collision>
+        <inertial>
+          <mass value="${bumper_m}"/>
+          <origin rpy="0 0 0" xyz="0 0 0"/>
+          <inertia ixx="${1/12*bumper_m*(bumper_y*bumper_y+bumper_z*bumper_z)}" ixy="0" ixz="0" iyy="${1/12*bumper_m*(bumper_z*bumper_z+bumper_x*bumper_x)}" iyz="0" izz="${1/12*bumper_m*(bumper_x*bumper_x+bumper_y*bumper_y)}"/>
+        </inertial>
+      </link>
+      <joint name="joint_chassis_rbumper" type="fixed">
+        <origin xyz="-${chassis_x/2} 0 ${(chassis_z+base_z)/2-chassis_z/2}" rpy="0 0 0"/>
+        <parent link="link_chassis"/>
+        <child link="link_rbumper"/>
+      </joint>
+      <link name="link_rbumper">
+        <visual>
+          <origin xyz="-${bumper_x/2} 0 0" rpy="0 0 0" />
+          <geometry>
+            <box size="${bumper_x} ${bumper_y} ${bumper_z}"/>
+          </geometry>
+        </visual>
+        <collision>
+          <origin xyz="-${bumper_x/2} 0 0" rpy="0 0 0" />
+          <geometry>
+            <box size="${bumper_x} ${bumper_y} ${bumper_z}"/>
+          </geometry>
+        </collision>
+        <inertial>
+          <mass value="${bumper_m}"/>
+          <origin rpy="0 0 0" xyz="0 0 0"/>
+          <inertia ixx="${1/12*bumper_m*(bumper_y*bumper_y+bumper_z*bumper_z)}" ixy="0" ixz="0" iyy="${1/12*bumper_m*(bumper_z*bumper_z+bumper_x*bumper_x)}" iyz="0" izz="${1/12*bumper_m*(bumper_x*bumper_x+bumper_y*bumper_y)}"/>
         </inertial>
       </link>

File: dor_description/urdf/laser.urdf.xacro (robot description, xacro)
@@ -16,5 +16,5 @@
           <origin xyz="0 0 0" rpy="0 0 0"/>
           <geometry>
-            <box size="0.1 0.1 0.1"/>
+            <box size="0.05 0.05 0.05"/>
           </geometry>
         </collision>
@@ -22,5 +22,5 @@
           <origin xyz="0 0 0" rpy="0 0 0"/>
           <geometry>
-            <box size="0.1 0.1 0.1"/>
+            <box size="0.05 0.05 0.05"/>
           </geometry>
         </visual>
@@ -33,5 +33,5 @@
       <!-- hokuyo -->
       <gazebo reference="link_hokuyo">
-        <material>Gazebo/Orange</material>
+        <material>Gazebo/Blue</material>
         <sensor type="gpu_ray" name="head_hokuyo_sensor">
           <pose>0 0 0 0 0 0</pose>

File: dor_description/urdf/mobile_robot.urdf.xacro (robot description, xacro)
@@ -2,37 +2,23 @@
 <robot name="mobile_robot" xmlns:xacro="https://www.ros.org/wiki/xacro" >
     <xacro:include filename="$(find dor_description)/urdf/fourwheeler.urdf.xacro" />
-    <xacro:fourwheeler_base_macro>
-      <xacro:property name="chassis_x" value="0.6" />
-      <xacro:property name="chassis_y" value="0.4" />
-      <xacro:property name="chassis_z" value="0.2" />
-      <xacro:property name="support_x" value="0.6" />
-      <xacro:property name="support_y" value="0.4" />
-      <xacro:property name="support_z" value="0.6" />
-      <xacro:property name="wheel_r" value="0.15"/>
-      <xacro:property name="wheel_l" value="0.08"/>
-      <xacro:property name="wheelbase" value="0.4" />
-      <xacro:property name="track" value="0.48" />
-    </xacro:fourwheeler_base_macro>
+    <xacro:fourwheeler_base_macro/>
+    <!--mobile base 50 cm x 50 cm square-->
     <xacro:include filename="$(find dor_description)/urdf/operate_device.urdf.xacro" />
     <xacro:operate_device_macro parent="link_support" robotname="mobile_robot">
-      <xacro:property name="location_x" value="0.3" />
+      <xacro:property name="location_x" value="0.25" />
       <xacro:property name="location_y" value="0" />
       <xacro:property name="location_z" value="0.5" />
     </xacro:operate_device_macro>
     <xacro:include filename="$(find dor_description)/urdf/camera.urdf.xacro"/>
-    <xacro:camera_macro parent="link_support">
-      <xacro:property name="location_x" value="0.2" />
-      <xacro:property name="location_y" value="0" />
-      <xacro:property name="location_z" value="0.3" />
-      <xacro:property name="support_x" value="0.02"/>
-      <xacro:property name="support_y" value="0.02"/>
-      <xacro:property name="support_z" value="0.8"/>
-      <xacro:property name="support_m" value="0.5"/>
+    <xacro:camera_macro parent="link_bar">
+      <xacro:property name="location_x" value="0.025" />
+      <xacro:property name="location_y" value="0.0" />
+      <xacro:property name="location_z" value="0.5" />
     </xacro:camera_macro>
     <xacro:include filename="$(find dor_description)/urdf/laser.urdf.xacro"/>
-    <xacro:laser_macro parent="link_chassis">
-      <xacro:property name="location_x" value="0.35" />
+    <xacro:laser_macro parent="link_support">
+      <xacro:property name="location_x" value="0.275" />
       <xacro:property name="location_y" value="0" />
-      <xacro:property name="location_z" value="0" />
+      <xacro:property name="location_z" value="-0.1" />
     </xacro:laser_macro>
 </robot>

File: dor_description/urdf/operate_device.urdf.xacro (robot description, xacro)
@@ -4,5 +4,17 @@
     <xacro:property name="location_x" value="0.25" />
     <xacro:property name="location_y" value="0" />
-    <xacro:property name="location_z" value="0.3" />
+    <xacro:property name="location_z" value="0.5" />
+    <xacro:property name="bar_x" value="0.02" />
+    <xacro:property name="bar_y" value="0.2" />
+    <xacro:property name="bar_z" value="1.0" />
+    <xacro:property name="bar_m" value="0.1" />
+    <xacro:property name="vslider_x" value="0.02" />
+    <xacro:property name="vslider_y" value="0.5" />
+    <xacro:property name="vslider_z" value="0.05" />
+    <xacro:property name="vslider_m" value="0.1" />
+    <xacro:property name="hslider_x" value="0.02" />
+    <xacro:property name="hslider_y" value="0.05" />
+    <xacro:property name="hslider_z" value="0.05" />
+    <xacro:property name="hslider_m" value="0.1" />
     <xacro:macro name="operate_device_macro" params="parent robotname">
       <joint name="joint_support_bar" type="fixed">
@@ -13,78 +25,78 @@
       <link name="link_bar">
         <visual>
-          <origin xyz="0.01 0 0" rpy="0 0 0" />
+          <origin xyz="${bar_x/2} 0 0" rpy="0 0 0" />
           <geometry>
-            <box size="0.02 0.3 0.02"/>
+            <box size="${bar_x} ${bar_y} ${bar_z}"/>
           </geometry>
         </visual>
         <collision>
-          <origin xyz="0.01 0 0" rpy="0 0 0" />
+          <origin xyz="${bar_x/2} 0 0" rpy="0 0 0" />
           <geometry>
-            <box size="0.02 0.3 0.02"/>
+            <box size="${bar_x} ${bar_y} ${bar_z}"/>
           </geometry>
         </collision>
         <inertial>
-          <mass value="0.01"/>
-          <origin xyz="0.01 0 0" rpy="0 0 0"/>
-          <inertia ixx="0.000034" ixy="0" ixz="0" iyy="0.00000067" iyz="0" izz="0.000034"/>
+          <mass value="${bar_m}"/>
+          <origin xyz="${bar_x/2} 0 0" rpy="0 0 0"/>
+          <inertia ixx="${1/12*bar_m*(bar_y*bar_y+bar_z*bar_z)}" ixy="0" ixz="0" iyy="${1/12*bar_m*(bar_z*bar_z+bar_x*bar_x)}" iyz="0" izz="${1/12*bar_m*(bar_x*bar_x+bar_y*bar_y)}"/>
         </inertial>
       </link>
-      <!--joint name="joint_bar_slider1" type="prismatic" have an issue-->
-      <joint name="joint_bar_slider1" type="fixed">
-        <origin xyz="0.02 0 0" rpy="0 0 0"/>
+      <joint name="joint_bar_vslider" type="prismatic">
+        <origin xyz="${bar_x} 0 0" rpy="0 0 0"/>
         <parent link="link_bar"/>
-        <child link="link_slider1"/>
-        <axis xyz="0 1 0"/>
-        <limit upper="0.15" lower="-0.15" effort="100.0" velocity="0.1"/>
-        <dynamics damping="0" friction="0"/>
+        <child link="link_vslider"/>
+        <axis xyz="0 0 1"/>
+        <limit upper="0.9" lower="-0.4" effort="100.0" velocity="1.0"/>
+        <dynamics damping="1.0" friction="30.0"/>
       </joint>
-      <link name="link_slider1">
+      <link name="link_vslider">
         <visual>
-          <origin xyz="0.01 0 0" rpy="0 0 0" />
+          <origin xyz="${vslider_x/2} 0 0" rpy="0 0 0" />
           <geometry>
-            <box size="0.02 0.02 0.8"/>
+            <box size="${vslider_x} ${vslider_y} ${vslider_z}"/>
           </geometry>
         </visual>
         <collision>
-          <origin xyz="0.01 0 0" rpy="0 0 0" />
+          <origin xyz="${vslider_x/2} 0 0" rpy="0 0 0" />
           <geometry>
-            <box size="0.02 0.02 0.8"/>
+            <box size="${vslider_x} ${vslider_y} ${vslider_z}"/>
           </geometry>
         </collision>
         <inertial>
-          <mass value="0.02"/>
-          <origin xyz="0.01 0 0" rpy="0 0 0"/>
-          <inertia ixx="0.0006" ixy="0" ixz="0" iyy="0.0006" iyz="0" izz="0.00000013"/>
+          <mass value="${vslider_m}"/>
+          <origin xyz="${vslider_x/2} 0 0" rpy="0 0 0"/>
+          <inertia ixx="${1/12*vslider_m*(vslider_y*vslider_y+vslider_z*vslider_z)}" ixy="0" ixz="0" iyy="${1/12*vslider_m*(vslider_z*vslider_z+vslider_x*vslider_x)}" iyz="0" izz="${1/12*vslider_m*(vslider_x*vslider_x+vslider_y*vslider_y)}"/>
         </inertial>
       </link>
-      <joint name="joint_slider1_slider2" type="prismatic">
-        <origin xyz="0.02 0 0" rpy="0 0 0"/>
-        <parent link="link_slider1"/>
-        <child link="link_slider2"/>
-        <axis xyz="0 0 1"/>
-        <limit upper="0.38" lower="-0.38" effort="30.0" velocity="0.1"/>
+      <joint name="joint_slider_slider" type="fixed">
+        <origin xyz="${vslider_x} 0 0" rpy="0 0 0"/>
+        <parent link="link_vslider"/>
+        <child link="link_hslider"/>
+        <axis xyz="0 1 0"/>
+        <limit upper="0.225" lower="-0.225" effort="100.0" velocity="0.5"/>
+        <dynamics damping="1.0" friction="30.0"/>
       </joint>
-      <link name="link_slider2">
+      <link name="link_hslider">
         <visual>
-          <origin xyz="0.01 0 0" rpy="0 0 0" />
+          <origin xyz="${hslider_x/2} 0 0" rpy="0 0 0" />
           <geometry>
-            <box size="0.02 0.04 0.04"/>
+            <box size="${hslider_x} ${hslider_y} ${hslider_z}"/>
           </geometry>
         </visual>
         <collision>
-          <origin xyz="0.01 0 0" rpy="0 0 0" />
+          <origin xyz="${hslider_x/2} 0 0" rpy="0 0 0" />
           <geometry>
-            <box size="0.02 0.04 0.04"/>
+            <box size="${hslider_x} ${hslider_y} ${hslider_z}"/>
           </geometry>
         </collision>
         <inertial>
-          <mass value="0.02"/>
-          <origin xyz="0.01 0 0" rpy="0 0 0"/>
-          <inertia ixx="0.0006" ixy="0" ixz="0" iyy="0.0006" iyz="0" izz="0.00000013"/>
+          <mass value="${hslider_m}"/>
+          <origin xyz="${hslider_x/2} 0 0" rpy="0 0 0"/>
+          <inertia ixx="${1/12*hslider_m*(hslider_y*hslider_y+hslider_z*hslider_z)}" ixy="0" ixz="0" iyy="${1/12*hslider_m*(hslider_z*hslider_z+hslider_x*hslider_x)}" iyz="0" izz="${1/12*hslider_m*(hslider_x*hslider_x+hslider_y*hslider_y)}"/>
         </inertial>
       </link>
       <joint name="joint_slider_finger" type="fixed">
-        <origin xyz="0.02 0 0" rpy="0 0 0"/>
-        <parent link="link_slider2"/>
+        <origin xyz="${hslider_x} 0 0" rpy="0 0 0"/>
+        <parent link="link_hslider"/>
         <child link="link_finger"/>
       </joint>
@@ -132,32 +144,32 @@
         </inertial>
       </link>
-      <!--transmission name="bar_trans">
+      <transmission name="vertical_trans">
         <type>transmission_interface/SimpleTransmission</type>
-        <joint name="joint_bar_slider1">
+        <joint name="joint_bar_vslider">
           <hardwareInterface>EffortJointInterface</hardwareInterface>
         </joint>
-        <actuator name="bar_motor">
-          <hardwareInterface>EffortJointInterface</hardwareInterface>
-          <mechanicalReduction>1</mechanicalReduction>
-        </actuator>
-      </transmission-->
-      <transmission name="lift_trans">
-        <type>transmission_interface/SimpleTransmission</type>
-        <joint name="joint_slider1_slider2">
-          <hardwareInterface>EffortJointInterface</hardwareInterface>
-        </joint>
-        <actuator name="lift_motor">
+        <actuator name="vertical_motor">
           <hardwareInterface>EffortJointInterface</hardwareInterface>
           <mechanicalReduction>1</mechanicalReduction>
         </actuator>
       </transmission>
+      <!-- <transmission name="horizontal_trans">
+        <type>transmission_interface/SimpleTransmission</type>
+        <joint name="joint_slider_slider">
+          <hardwareInterface>EffortJointInterface</hardwareInterface>
+        </joint>
+        <actuator name="horizontal_motor">
+          <hardwareInterface>EffortJointInterface</hardwareInterface>
+          <mechanicalReduction>1</mechanicalReduction>
+        </actuator>
+      </transmission> -->
       <gazebo reference="link_bar">
         <material>Gazebo/Orange</material>
       </gazebo>
-      <gazebo reference="link_slider1">
+      <gazebo reference="link_vslider">
         <material>Gazebo/Orange</material>
       </gazebo>
-      <gazebo reference="link_slider2">
-        <material>Gazebo/Grey</material>
+      <gazebo reference="link_hslider">
+        <material>Gazebo/Orange</material>
       </gazebo>
       <gazebo>
