Commit message: add walloutlet and camera

File: dor_description/urdf/camera.urdf.xacro (robot description, xacro)
@@ -4,75 +4,69 @@
     <xacro:property name="location_x" value="0" />
     <xacro:property name="location_y" value="0" />
-    <xacro:property name="location_z" value="1.0" />
-    <xacro:property name="realsense_d435_width" value="0.09"/>
-    <xacro:property name="realsense_d435_height" value="0.025"/>
-    <xacro:property name="realsense_d435_depth" value="0.025"/>
-    <!-- Intel_RealSense_D400_Family_Datasheet_Jan2019.pdf, page 64 -->
-    <xacro:property name="realsense_d435_front_to_depth" value="0.0042" />
-    <!-- Measured from CAD file -->
-    <xacro:property name="realsense_d435_mount_hole_to_front" value="0.0149" />
-    <xacro:property name="realsense_d435_case_offset_x" value="${realsense_d435_front_to_depth - realsense_d435_depth/2.0}"/>
-    <!-- mounting hole to depth frame, Intel_RealSense_D400_Family_Datasheet_Jan2019.pdf, page 66 -->
-    <xacro:property name="realsense_d435_case_offset_y" value="-0.0175"/>
-    <xacro:property name="realsense_d435_case_offset_z" value="0.0"/>
+    <xacro:property name="location_z" value="0" />
+    <xacro:property name="camera_link" value="0.02" />
     <xacro:macro name="camera_macro" params="parent">
-      <!--camera-->
-      <joint name="joint_rs435" type="fixed">
-        <origin xyz="${location_x+realsense_d435_depth/2.0} ${location_y} ${location_z}" rpy="0 0 0"/>
-        <parent link="${parent}"/>
-        <child link="link_rs435"/>
-      </joint>
-      <link name="link_rs435">
-        <inertial>
-          <mass value="0.072" />
-          <origin xyz="0 0 0" rpy="0 0 0" />
-          <inertia ixx="5.8083e-4" ixy="0" ixz="0" iyy="3.0833e-5" iyz="0" izz="5.9083e-4" />
-          <inertia ixx="1.0e-6" ixy="0" ixz="0" iyy="1.0e-6" iyz="0" izz="1.0e-6" />
-        </inertial>
-        <visual>
-          <origin xyz="${realsense_d435_front_to_depth} ${realsense_d435_case_offset_y} 0.0" rpy="${M_PI/2} 0 ${M_PI/2}" />
-          <geometry>
-            <mesh filename="package://dor_description/meshes/intel_realsense_d435/D435.dae" scale="0.001 0.001 0.001" />
-          </geometry>
-        </visual>
-        <collision>
-          <origin xyz="${realsense_d435_case_offset_x} ${realsense_d435_case_offset_y} ${realsense_d435_case_offset_z}" rpy="0 0 0" />
-          <geometry>
-            <box size="${realsense_d435_depth} ${realsense_d435_width} ${realsense_d435_height}" />
-          </geometry>
-        </collision>
-      </link>
-      <!--gazebo plugin-->
-      <gazebo reference="link_rs435">
-        <material>Gazebo/Grey</material>
-        <sensor type="depth" name="rs435">
-          <update_rate>30</update_rate>
-          <camera>
-            <horizontal_fov>${69.4*M_PI/180.0}</horizontal_fov>
-            <vertical_fov>${42.5*M_PI/180.0}</vertical_fov>
-            <diagonal_fov>${77.0*M_PI/180.0}</diagonal_fov>
-            <image>
-              <format>B8G8R8</format>
-              <!-- <width>1280</width>
-              <height>720</height> -->
-              <width>640</width>
-              <height>480</height>
-            </image>
-            <clip>
-              <near>0.15</near>
-              <far>9.0</far>
-            </clip>
-          </camera>
-          <plugin name="rs435_camera_plugin" filename="libgazebo_ros_openni_kinect.so">
-            <cameraName>rs435</cameraName>
-            <imageTopicName>color/image_raw</imageTopicName>
-            <cameraInfoTopicName>color/camera_info</cameraInfoTopicName>
-            <depthImageTopicName>depth/image_raw</depthImageTopicName>
-            <depthImageCameraInfoTopicName>depth/camera_info</depthImageCameraInfoTopicName>
-            <pointCloudTopicName>depth/points</pointCloudTopicName>
-            <frameName>rs435_frame</frameName>
-          </plugin>
-        </sensor>
-      </gazebo>
+    <!--movable camera-->
+    <joint name="camera_joint" type="fixed">
+      <origin xyz="${location_x} ${location_y} ${location_z}" rpy="0 0 0"/>
+      <parent link="${parent}"/>
+      <child link="camera_link"/>
+    </joint>
+    <link name="camera_link">
+      <collision>
+        <origin xyz="0 0 ${camera_link/2}" rpy="0 0 0"/>
+        <geometry>
+          <box size="${camera_link} ${camera_link} ${camera_link}"/>
+        </geometry>
+      </collision>
+      <visual>
+        <origin xyz="0 0 ${camera_link/2}" rpy="0 0 0"/>
+        <geometry>
+          <box size="${camera_link} ${camera_link} ${camera_link}"/>
+        </geometry>
+      </visual>
+      <inertial>
+        <mass value="1e-5" />
+        <origin xyz="0 0 0" rpy="0 0 0"/>
+        <inertia ixx="1e-6" ixy="0" ixz="0" iyy="1e-6" iyz="0" izz="1e-6" />
+      </inertial>
+    </link>
+    <gazebo reference="camera_link">
+      <material>Gazebo/Red</material>
+      <sensor type="camera" name="camera_front">
+        <update_rate>30.0</update_rate>
+        <camera name="head">
+          <horizontal_fov>1.3962634</horizontal_fov>
+          <image>
+            <width>800</width>
+            <height>800</height>
+            <format>R8G8B8</format>
+          </image>
+          <clip>
+            <near>0.02</near>
+            <far>300</far>
+          </clip>
+          <noise>
+            <type>gaussian</type>
+            <mean>0.0</mean>
+            <stddev>0.007</stddev>
+          </noise>
+        </camera>
+        <plugin name="camera_controller" filename="libgazebo_ros_camera.so">
+          <alwaysOn>true</alwaysOn>
+          <updateRate>0.0</updateRate>
+          <cameraName>front_cam</cameraName>
+          <imageTopicName>image_raw</imageTopicName>
+          <cameraInfoTopicName>camera_info</cameraInfoTopicName>
+          <frameName>camera_link</frameName>
+          <hackBaseline>0.07</hackBaseline>
+          <distortionK1>0.0</distortionK1>
+          <distortionK2>0.0</distortionK2>
+          <distortionK3>0.0</distortionK3>
+          <distortionT1>0.0</distortionT1>
+          <distortionT2>0.0</distortionT2>
+        </plugin>
+      </sensor>
+    </gazebo>
     </xacro:macro>
 </robot>

File: dor_description/urdf/mobile_robot.urdf.xacro (robot description, xacro)
@@ -10,9 +10,15 @@
       <xacro:property name="location_z" value="0.55" />
     </xacro:operate_device_macro>
-    <xacro:include filename="$(find dor_description)/urdf/camera.urdf.xacro"/>
-    <xacro:camera_macro parent="link_bar">
+    <xacro:include filename="$(find dor_description)/urdf/realsense.urdf.xacro"/>
+    <xacro:realsense_macro parent="link_bar">
       <xacro:property name="location_x" value="0.025" />
       <xacro:property name="location_y" value="0.0" />
       <xacro:property name="location_z" value="0.5" />
+    </xacro:realsense_macro>
+    <xacro:include filename="$(find dor_description)/urdf/camera.urdf.xacro"/>
+    <xacro:camera_macro parent="link_finger">
+      <xacro:property name="location_x" value="0.1" />
+      <xacro:property name="location_y" value="0.0" />
+      <xacro:property name="location_z" value="0.01" />
     </xacro:camera_macro>
     <xacro:include filename="$(find dor_description)/urdf/laser.urdf.xacro"/>

File: dor_description/urdf/operate_device.urdf.xacro (robot description, xacro)
@@ -58,5 +58,5 @@
         <child link="link_vslider"/>
         <axis xyz="0 0 1"/>
-        <limit upper="${bar_z-0.05}" lower="0.0" effort="1000.0" velocity="0.5"/>
+        <limit upper="${bar_z-0.05}" lower="0.05" effort="1000.0" velocity="0.5"/>
         <dynamics damping="0" friction="1.0"/>
       </joint>

Commit message: add door opening trainer

File: dor_description/urdf/camera.urdf.xacro (robot description, xacro)
@@ -5,9 +5,14 @@
     <xacro:property name="location_y" value="0" />
     <xacro:property name="location_z" value="0" />
+    <xacro:property name="location_r" value="0" />
+    <xacro:property name="location_p" value="0" />
+    <xacro:property name="location_y" value="0" />
+    <xacro:property name="camera_width" value="800" />
+    <xacro:property name="camera_height" value="800" />
     <xacro:property name="camera_link" value="0.02" />
     <xacro:macro name="camera_macro" params="parent">
     <!--movable camera-->
     <joint name="camera_joint" type="fixed">
-      <origin xyz="${location_x} ${location_y} ${location_z}" rpy="0 0 0"/>
+      <origin xyz="${location_x} ${location_y} ${location_z}" rpy="${location_r} ${location_p} ${location_y}"/>
       <parent link="${parent}"/>
       <child link="camera_link"/>
@@ -39,6 +44,6 @@
           <horizontal_fov>1.3962634</horizontal_fov>
           <image>
-            <width>800</width>
-            <height>800</height>
+            <width>${camera_width}</width>
+            <height>${camera_height}</height>
             <format>R8G8B8</format>
           </image>

Commit message: add reinforcement learning environment

File: dor_description/urdf/camera.urdf.xacro (robot description, xacro)
@@ -8,6 +8,6 @@
     <xacro:property name="location_p" value="0" />
     <xacro:property name="location_y" value="0" />
-    <xacro:property name="camera_width" value="800" />
-    <xacro:property name="camera_height" value="800" />
+    <xacro:property name="camera_width" value="600" />
+    <xacro:property name="camera_height" value="600" />
     <xacro:property name="camera_link" value="0.02" />
     <xacro:macro name="camera_macro" params="parent">

Commit message: add two more cameras

File: dor_description/urdf/camera.urdf.xacro (robot description, xacro)
@@ -11,12 +11,13 @@
     <xacro:property name="camera_height" value="600" />
     <xacro:property name="camera_link" value="0.02" />
+    <xacro:property name="camera_name" value="front_cam" />
     <xacro:macro name="camera_macro" params="parent">
     <!--movable camera-->
-    <joint name="camera_joint" type="fixed">
+    <joint name="camera_joint_${camera_name}" type="fixed">
       <origin xyz="${location_x} ${location_y} ${location_z}" rpy="${location_r} ${location_p} ${location_y}"/>
       <parent link="${parent}"/>
-      <child link="camera_link"/>
+      <child link="camera_link_${camera_name}"/>
     </joint>
-    <link name="camera_link">
+    <link name="camera_link_${camera_name}">
       <collision>
         <origin xyz="0 0 ${camera_link/2}" rpy="0 0 0"/>
@@ -37,7 +38,7 @@
       </inertial>
     </link>
-    <gazebo reference="camera_link">
+    <gazebo reference="camera_link_${camera_name}">
       <material>Gazebo/Red</material>
-      <sensor type="camera" name="camera_front">
+      <sensor type="camera" name="${camera_name}">
         <update_rate>30.0</update_rate>
         <camera name="head">
@@ -61,8 +62,8 @@
           <alwaysOn>true</alwaysOn>
           <updateRate>0.0</updateRate>
-          <cameraName>front_cam</cameraName>
+          <cameraName>${camera_name}</cameraName>
           <imageTopicName>image_raw</imageTopicName>
           <cameraInfoTopicName>camera_info</cameraInfoTopicName>
-          <frameName>camera_link</frameName>
+          <frameName>${camera_name}</frameName>
           <hackBaseline>0.07</hackBaseline>
           <distortionK1>0.0</distortionK1>

File: dor_description/urdf/realsense.urdf.xacro (robot description, xacro)
@@ -16,4 +16,5 @@
     <xacro:property name="realsense_d435_case_offset_y" value="-0.0175"/>
     <xacro:property name="realsense_d435_case_offset_z" value="0.0"/>
+    <xacro:property name="topic" value="rs435">
     <xacro:macro name="realsense_macro" params="parent">
       <!--camera-->
@@ -65,5 +66,5 @@
           </camera>
           <plugin name="rs435_camera_plugin" filename="libgazebo_ros_openni_kinect.so">
-            <cameraName>rs435</cameraName>
+            <cameraName>${topic}</cameraName>
             <imageTopicName>color/image_raw</imageTopicName>
             <cameraInfoTopicName>color/camera_info</cameraInfoTopicName>

File: dor_description/urdf/training_mobile_robot.urdf.xacro (robot description, xacro)
@@ -14,4 +14,5 @@
       <xacro:property name="camera_width" value="600" />
       <xacro:property name="camera_height" value="600" />
+      <xacro:property name="camera_name" value="cam_up"/>
     </xacro:camera_macro>
 </robot>
