Commit message: reset the envrionment of door opening training

File: dor_description/urdf/fourwheeler_base.urdf.xacro (robot description, xacro)
@@ -234,5 +234,5 @@
       <!--hook for opening door-->
       <joint name="joint_fbummer_hook" type="fixed">
-        <origin xyz="${bumper_x/2} ${bumper_y/2} ${bumper_z/2}" rpy="0 0 0"/>
+        <origin xyz="${bumper_x/2} -${bumper_y/2} ${bumper_z/2}" rpy="0 0 0"/>
         <parent link="link_fbumper"/>
         <child link="link_hook"/>
@@ -264,5 +264,5 @@
       <link name="link_tip">
         <visual>
-          <origin xyz="${tip_x/2} -0.02 ${tip_z/2}" rpy="0 0 0" />
+          <origin xyz="${tip_x/2} 0.02 ${tip_z/2}" rpy="0 0 0" />
           <geometry>
             <box size="${tip_x} ${tip_y} ${tip_z}"/>
@@ -270,5 +270,5 @@
         </visual>
         <collision>
-          <origin xyz="${tip_x/2} -0.02 ${tip_z/2}" rpy="0 0 0" />
+          <origin xyz="${tip_x/2} 0.02 ${tip_z/2}" rpy="0 0 0" />
           <geometry>
             <box size="${tip_x} ${tip_y} ${tip_z}"/>

Commit message: add force sensor

File: dor_description/urdf/fourwheeler_base.urdf.xacro (robot description, xacro)
@@ -257,6 +257,8 @@
         </inertial>
       </link>
-      <joint name="joint_hook_tip" type="fixed">
+      <joint name="joint_hook_tip" type="revolute">
+        <axis xyz="0 0 1" rpy="0 0 0"/>
         <origin xyz="${hook_x} ${hook_y/2} 0" rpy="0 0 0"/>
+        <limit velocity="0.0" effort="100" lower="0" upper="0"/>
         <parent link="link_hook"/>
         <child link="link_tip"/>
@@ -318,21 +320,21 @@
       </gazebo>
       <gazebo reference="link_lrwheel">
-        <mu1>0.1</mu1>
-        <mu2>0.1</mu2>
+        <mu1>0.99</mu1>
+        <mu2>0.99</mu2>
         <material>Gazebo/Black</material>
       </gazebo>
       <gazebo reference="link_rrwheel">
-        <mu1>0.1</mu1>
-        <mu2>0.1</mu2>
+        <mu1>0.99</mu1>
+        <mu2>0.99</mu2>
         <material>Gazebo/Black</material>
       </gazebo>
       <gazebo reference="link_lfwheel">
-        <mu1>0.1</mu1>
-        <mu2>0.1</mu2>
+        <mu1>0.99</mu1>
+        <mu2>0.99</mu2>
         <material>Gazebo/Black</material>
       </gazebo>
       <gazebo reference="link_rfwheel">
-        <mu1>0.1</mu1>
-        <mu2>0.1</mu2>
+        <mu1>0.99</mu1>
+        <mu2>0.99</mu2>
         <material>Gazebo/Black</material>
       </gazebo>
@@ -342,4 +344,20 @@
       <gazebo reference="link_tip">
         <material>Gazebo/Black</material>
+      </gazebo>
+      <!--ft force sensor in joint-->
+      <gazebo reference ="joint_hook_tip">
+        <provideFeedback>true</provideFeedback>
+      </gazebo>
+      <gazebo>
+        <plugin name="ft_sensor" filename="libgazebo_ros_ft_sensor.so">
+          <updateRate>100.0</updateRate>
+          <topicName>tf_sensor_topic</topicName>
+          <jointName>joint_hook_tip</jointName>
+          <noise>
+            <type>guassian</type>
+            <mean>0.0</mean>
+            <stddev>0.003</stddev>
+          </noise>
+        </plugin>
       </gazebo>
     </xacro:macro>

Commit message: add force sensor

File: dor_description/urdf/fourwheeler_base.urdf.xacro (robot description, xacro)
@@ -233,5 +233,7 @@
       </link>
       <!--hook for opening door-->
-      <joint name="joint_fbummer_hook" type="fixed">
+      <joint name="joint_fbummer_hook" type="revolute">
+        <axis xyz="1 0 0" rpy="0 0 0"/>
+        <limit velocity="0" effort="1000" lower="0" upper="0"/>
         <origin xyz="${bumper_x/2} -${bumper_y/2} ${bumper_z/2}" rpy="0 0 0"/>
         <parent link="link_fbumper"/>
@@ -257,8 +259,6 @@
         </inertial>
       </link>
-      <joint name="joint_hook_tip" type="revolute">
-        <axis xyz="0 0 1" rpy="0 0 0"/>
+      <joint name="joint_hook_tip" type="fixed">
         <origin xyz="${hook_x} ${hook_y/2} 0" rpy="0 0 0"/>
-        <limit velocity="0.0" effort="100" lower="0" upper="0"/>
         <parent link="link_hook"/>
         <child link="link_tip"/>
@@ -320,21 +320,21 @@
       </gazebo>
       <gazebo reference="link_lrwheel">
-        <mu1>0.99</mu1>
-        <mu2>0.99</mu2>
+        <mu1>0.8</mu1>
+        <mu2>0.8</mu2>
         <material>Gazebo/Black</material>
       </gazebo>
       <gazebo reference="link_rrwheel">
-        <mu1>0.99</mu1>
-        <mu2>0.99</mu2>
+        <mu1>0.8</mu1>
+        <mu2>0.8</mu2>
         <material>Gazebo/Black</material>
       </gazebo>
       <gazebo reference="link_lfwheel">
-        <mu1>0.99</mu1>
-        <mu2>0.99</mu2>
+        <mu1>0.8</mu1>
+        <mu2>0.8</mu2>
         <material>Gazebo/Black</material>
       </gazebo>
       <gazebo reference="link_rfwheel">
-        <mu1>0.99</mu1>
-        <mu2>0.99</mu2>
+        <mu1>0.8</mu1>
+        <mu2>0.8</mu2>
         <material>Gazebo/Black</material>
       </gazebo>
@@ -346,5 +346,5 @@
       </gazebo>
       <!--ft force sensor in joint-->
-      <gazebo reference ="joint_hook_tip">
+      <gazebo reference ="joint_fbummer_hook">
         <provideFeedback>true</provideFeedback>
       </gazebo>
@@ -353,5 +353,5 @@
           <updateRate>100.0</updateRate>
           <topicName>tf_sensor_topic</topicName>
-          <jointName>joint_hook_tip</jointName>
+          <jointName>joint_fbummer_hook</jointName>
           <noise>
             <type>guassian</type>
